File: hardware/kicad/mainboard/mainboard.kicad_sch (KiCad schematic)
At the start: 17 parts, among them J1 230 VAC in, J2 24 VAC to relay COMs / valve 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, SW1 CONFIG (GPIO 23), T1 Transformer_1P_1S

Commit message: connect what it needed
Parts:
- added B1: 3.7V LiPo, symbol Device:Battery_Cell
- added J3: A1 on-board JST PH2.0 BAT socket, symbol Connector_Generic:Conn_01x02
- R1: value 4.7k -> 3.3k
- R5: value 3.3k -> 4.7k
Connections:
- net +3V3: now also R5.1; no longer A1.17 (3V3), R1.1
- net GND: now also R1.2; no longer A1.15 (GND), R5.2
- net I2C_SCL: no longer A1.10 (SCL_IO20)
- net I2C_SDA: no longer A1.9 (SDA_IO19)
- net ONEWIRE: now also R5.2; no longer R1.2
- net PRESS_ADC: now also R1.1, R2.1; no longer R2.2, R3.1
- net WIND_ADC: now also R3.1, R4.1; no longer R4.2, R5.1
- net PRESS_OUT: no longer names the net of A5.3 (OUT)
- net PRESS_OUT: now also R2.2; no longer R2.1
- net WIND_OUT: no longer names the net of A6.3 (OUT)
- net WIND_OUT: now also R4.2; no longer R4.1
- new net BAT+: B1.1 (+), J3.1 (Pin_1)
- new net BAT-: B1.2 (-), J3.2 (Pin_2)
- no-connect marks 8 -> 12
Other:
- note added: "Power entry: +5V from an external 5 V supply, +24V for the wind sensor (10-30 V), +3V3 from the FireBeetle regulator. PWR_FLAGs mark the external sources. B1 plugs into the FireBeetle's own battery socket (J3 is that socket, not a separate part)."
- note removed: "Power entry: +5V from an external 5 V supply, +24V for the wind sensor (10-30 V), +3V3 from the FireBeetle regulator. PWR_FLAGs mark the external sources."
- moved on the sheet: A1, A2, A3, A4, A5, A6, A7, A8, T1

Commit message: connect the Power
Parts:
- removed T1: Transformer_1P_1S, symbol Device:Transformer_1P_1S
- added BT1, BT2: 12V SLA, symbol Device:Battery
- added C1: 10uF 50V, Capacitor_THT:CP_Radial_D6.3mm_P2.50mm, symbol Device:C
- added C2: 22uF, Capacitor_THT:CP_Radial_D6.3mm_P2.50mm, symbol Device:C
- added C3: 100nF 50V, Capacitor_THT:CP_Radial_D6.3mm_P2.50mm, symbol Device:C
- added F1: 1A, Fuse:Fuseholder_Cylinder-5x20mm_Stelvio-Kontek_PTF78_Horizontal_Open, symbol Device:Fuse
- added F2: 5A, Fuse:Fuseholder_Cylinder-5x20mm_Stelvio-Kontek_PTF78_Horizontal_Open, symbol Device:Fuse
- added F3: 1.5A, Fuse:Fuseholder_Cylinder-5x20mm_Stelvio-Kontek_PTF78_Horizontal_Open, symbol Device:Fuse
- added PS1: PSU_ACDC_27V6, libraries:PSU_ACDC_27V6, symbol FullModules:PSU_ACDC_27V6
- added R6: 100, Resistor_THT:R_Axial_DIN0207_L6.3mm_D2.5mm_P7.62mm_Horizontal, symbol Device:R
- added U1: R-78B5.0-2.0, Converter_DCDC:Converter_DCDC_RECOM_R-78B-2.0_THT, symbol Regulator_Switching:R-78B5.0-2.0
- added U2: LVD_Module_24V, libraries:LVD_Module_24V, symbol FullModules:LVD_Module_24V
- added U3: DCAC_Converter_24VAC, libraries:DCAC_Converter_24VAC, symbol FullModules:DCAC_Converter_24VAC
Connections:
- net +24V: now also C1.1, F3.1, PS1.3 (V+), U1.1 (IN), U2.3 (LOAD+)
- net +5V: now also C2.1, U1.3 (OUT)
- net GND: now also BT1.2 (-), C1.2, C2.2, PS1.4 (V-), U1.2 (GND), U2.2 (BAT-), U2.4 (LOAD-), U3.2 (VIN-)
- net at J1.2 (Pin_2): now also F1.1
- net at J1.1 (Pin_1): now also PS1.2 (N)
- net VAC24_B: now reaches J2.2 (Pin_2)
- net VAC24_B: now also C3.2, U3.5 (AC2)
- net VAC24_A: now reaches J2.1 (Pin_1)
- net VAC24_A: now also R6.1, U3.4 (AC1)
- new net: F1.2, PS1.1 (L)
- new net: F3.2, U3.1 (VIN+)
- new net: C3.1, R6.2
- new net: BT2.1 (+), F2.1
- new net: F2.2, U2.1 (BAT+)
- new net: BT1.1 (+), BT2.2 (-)
- no-connect marks 12 -> 13
Other:
- note added: "+3V3 comes from the FireBeetle regulator (PWR_FLAG). B1 plugs into the FireBeetle's own battery socket (J3 is that socket, not a separate part)."
- note removed: "Power entry: +5V from an external 5 V supply, +24V for the wind sensor (10-30 V), +3V3 from the FireBeetle regulator. PWR_FLAGs mark the external sources. B1 plugs into the FireBeetle's own battery socket (J3 is that socket, not a separate part)."

Commit message: add reserved for S3
Parts:
- added J4: S3 link, Connector_PinHeader_2.54mm:PinHeader_1x03_P2.54mm_Vertical, symbol Connector_Generic:Conn_01x03
Connections:
- net GND: now also J4.3 (Pin_3)
- net S3_TX: now reaches A1.20 (D11_IO7_INT)
- net S3_TX: now also J4.1 (Pin_1)
- net S3_RX: now reaches A1.21 (D12_IO6_TCS)
- net S3_RX: now also J4.2 (Pin_2)
- no-connect marks 13 -> 11
Other:
- note added: "NOTES - Valve GPIOs come from CONFIG_DYNAMIC_VALVE_GPIO_LIST = 1,14,18,21,22,16,17,5 (valves 1-8, CONFIG_DEVICE_MAX_VALVES = 8). All 8 relay channels are valves. - GPIO 16/17 are UART0: the console runs on USB Serial/JTAG. - No safe GPIO is left: more valves, the 24 VAC converter enable, mains-detect and battery sense need an I2C expander / I2C ADC. - Relay contacts are not in the relay module sy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"
- note removed: "NOTES - Valve GPIOs come from CONFIG_DYNAMIC_VALVE_GPIO_LIST = 1,14,18,21,22,16,17,5 (valves 1-8, CONFIG_DEVICE_MAX_VALVES = 8). All 8 relay channels are valves. - GPIO 16/17 are UART0: the console runs on USB Serial/JTAG. - No safe GPIO is left: more valves, the 24 VAC converter enable, mains-detect, battery sense and the LCD need an I2C expander / I2C ADC. - Relay contacts are not in the relay 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"
